File: hardware/projects/dolphin/dolphin.kicad_sch (KiCad schematic)
At the start: 0 parts

Commit message: refactor: add PCB views to SCH
Other:
- note added: "Block Diagram"
- note added: "bottom view"
- note added: "top view"
