File: hardware/projects/encoder/encoder.kicad_sch (KiCad schematic)
At the start: 19 parts

Commit message: refactor: add PCB views to SCH
Other:
- note added: "Diagram"
- note added: "bottom view"
- note added: "top view"
- moved on the sheet: C1, C2, E1, JP1, R1, R2, R3, TP1, TP10, TP11, TP12, TP2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
