File: hardware/projects/mainboard/led.kicad_sch (KiCad schematic)
At the start: 13 parts, among them J2 LRGB

Commit message: chore: rename schematic sheets
Other:
- title: dolphin -> dolphin/mainboard/led
Changed lines of the file:
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@@
 	(paper "A4")
 	(title_block
-		(title "dolphin")
+		(title "dolphin/mainboard/led")
 		(date "2026-08-03")
 		(rev "v2")
