File: hardware/projects/mainboard/mainboard.kicad_pcb (KiCad board)
At the start: 2 copper layers, 55 x 70 mm, 96 parts, among them J1 MICRO_START, J2 LRGB, J3 ESC_L, J4 Conn_02x08_Odd_Even, J7 ESC_R, J8 ENC_R, J9 ENC_L, P1 USB_C, SW1 SW_Push, U2 KF33BDT, U3 CD74HC4067M, U4 ESP32-S3-WROOM-1

Commit message: chore: rename schematic sheets
Other:
- board text added: "dolphin/mainboard_v2"
- board text removed: "dolphin_v2"
Changed lines of the file:
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@@
 		)
 	)
-	(gr_text "dolphin_v2\n"
+	(gr_text "dolphin/mainboard_v2\n"
 		(at 135.5 88.5 0)
 		(layer "F.SilkS")
