File: hardware/projects/mainboard/power.kicad_sch (KiCad schematic)
At the start: 14 parts, among them J1 MICRO_START, J3 ESC_L, J4 Conn_02x08_Odd_Even, J7 ESC_R, SW1 SW_Push, U4 ESP32-S3-WROOM-1

Commit message: chore: rename mainboard files
Parts:
- removed C10, C9: 1u, Capacitor_SMD:C_0805_2012Metric_Pad1.18x1.45mm_HandSolder, symbol Device:C
- removed J1: MICRO_START, dolphin:Connector_JST_ZH_B3B-ZR_1x03_P1.50mm_Vertical, symbol Connector_Generic:Conn_01x03
- removed J3: ESC_L, Connector_PinSocket_2.54mm:PinSocket_1x03_P2.54mm_Vertical, symbol Connector_Generic:Conn_01x03
- removed J4: Conn_02x08_Odd_Even, Connector_PinSocket_2.54mm:PinSocket_2x08_P2.54mm_Vertical, symbol Connector_Generic:Conn_02x08_Odd_Even
- removed J7: ESC_R, Connector_PinSocket_2.54mm:PinSocket_1x03_P2.54mm_Vertical, symbol Connector_Generic:Conn_01x03
- removed R22, R23, R25, R26, R27: 10k, Resistor_SMD:R_0805_2012Metric_Pad1.20x1.40mm_HandSolder, symbol Device:R_US
- removed R24: 20k, Resistor_SMD:R_0805_2012Metric_Pad1.20x1.40mm_HandSolder, symbol Device:R_US
- removed SW1: SW_Push, Button_Switch_SMD:SW_SPST_PTS810, symbol Switch:SW_Push
- removed U4: ESP32-S3-WROOM-1, dolphin:ESP32-S3-WROOM-1, symbol RF_Module:ESP32-S3-WROOM-1
- added C2, C3: 1u, Capacitor_SMD:C_0805_2012Metric_Pad1.18x1.45mm_HandSolder, symbol Device:C
- added C4, C5: 10u 16V, Capacitor_THT:CP_Radial_D5.0mm_P2.00mm, symbol Device:C_Polarized_US
- added D1, D2, D3: BLUE_2V6, LED_SMD:LED_0805_2012Metric_Pad1.15x1.40mm_HandSolder, symbol Device:LED
- added D4, D5: LESD5D5.0CT1G, Diode_SMD:D_0805_2012Metric_Pad1.15x1.40mm_HandSolder, symbol Device:D
- added H1, H2, H3, H4: M3, MountingHole:MountingHole_3.2mm_M3_Pad_Via, symbol Mechanical:MountingHole_Pad
- added P1: USB_C, dolphin:Connector_USB-C, symbol dolphin:Connector_USB-C
- added R16, R17, R18: 10k, Resistor_SMD:R_0805_2012Metric_Pad1.20x1.40mm_HandSolder, symbol Device:R_US
- added TP2: +BATT, TestPoint:TestPoint_Pad_D1.0mm, symbol Connector:TestPoint
- added TP3: 5V, TestPoint:TestPoint_Pad_D1.0mm, symbol Connector:TestPoint
- added TP4: 3V3, TestPoint:TestPoint_Pad_D1.0mm, symbol Connector:TestPoint
- added U1: (no value), dolphin:Regulator_DC-DC_MINI-360, symbol dolphin:Regulator_DC-DC_MINI-360
- added U2: KF33BDT, dolphin:Regulator_KF33BD-TR, symbol Regulator_Linear:KF33BDT
Connections:
- net +3V3: now also C3.1, C5.1, R17.1, TP4.1, U2.3 (VO)
- net +5V: now also C2.1, C4.1, P1.4 (VBUS), R16.1, TP3.1, U1.3 (VOUT), U2.1 (VI)
- net GND: now also C2.2, C3.2, C4.2, C5.2, D1.1 (K), D2.1 (K), D3.1 (K), D4.2 (A), D5.2 (A), H1.1, H2.1, H3.1, H4.1, P1.1 (GND), U1.2 (GND), U2.2 (GND)
- net USB_D+: now also D4.1 (K), P1.2 (D+)
- net USB_D-: now also D5.1 (K), P1.3 (D-)
- new net +BATT: R18.1, TP2.1, U1.1 (VIN)
- new net LED_3V3: D3.2 (A), R17.2
- new net LED_5V: D2.2 (A), R16.2
- new net LED_BATT: D1.2 (A), R18.2
- no-connect marks 5 -> 0
Other:
- note removed: "booting circuit"
- note removed: "decoupling"
- note removed: "resetting circuit"

Commit message: chore: rename schematic sheets
Other:
- title: dolphin -> dolphin/mainboard/power
Changed lines of the file:
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@@
 	(paper "A4")
 	(title_block
-		(title "dolphin")
+		(title "dolphin/mainboard/power")
 		(date "2026-08-03")
 		(rev "v2")
