File: hardware/projects/mainboard/processor.kicad_sch (KiCad schematic)
At the start: 22 parts, among them P1 USB_C, U2 KF33BDT

Commit message: chore: rename mainboard files
Parts:
- removed C2, C3: 1u, Capacitor_SMD:C_0805_2012Metric_Pad1.18x1.45mm_HandSolder, symbol Device:C
- removed C4, C5: 10u 16V, Capacitor_THT:CP_Radial_D5.0mm_P2.00mm, symbol Device:C_Polarized_US
- removed D1, D2, D3: BLUE_2V6, LED_SMD:LED_0805_2012Metric_Pad1.15x1.40mm_HandSolder, symbol Device:LED
- removed D4, D5: LESD5D5.0CT1G, Diode_SMD:D_0805_2012Metric_Pad1.15x1.40mm_HandSolder, symbol Device:D
- removed H1, H2, H3, H4: M3, MountingHole:MountingHole_3.2mm_M3_Pad_Via, symbol Mechanical:MountingHole_Pad
- removed P1: USB_C, dolphin:Connector_USB-C, symbol dolphin:Connector_USB-C
- removed R16, R17, R18: 10k, Resistor_SMD:R_0805_2012Metric_Pad1.20x1.40mm_HandSolder, symbol Device:R_US
- removed TP2: +BATT, TestPoint:TestPoint_Pad_D1.0mm, symbol Connector:TestPoint
- removed TP3: 5V, TestPoint:TestPoint_Pad_D1.0mm, symbol Connector:TestPoint
- removed TP4: 3V3, TestPoint:TestPoint_Pad_D1.0mm, symbol Connector:TestPoint
- removed U1: (no value), dolphin:Regulator_DC-DC_MINI-360, symbol dolphin:Regulator_DC-DC_MINI-360
- removed U2: KF33BDT, dolphin:Regulator_KF33BD-TR, symbol Regulator_Linear:KF33BDT
- added C10, C9: 1u, Capacitor_SMD:C_0805_2012Metric_Pad1.18x1.45mm_HandSolder, symbol Device:C
- added J1: MICRO_START, dolphin:Connector_JST_ZH_B3B-ZR_1x03_P1.50mm_Vertical, symbol Connector_Generic:Conn_01x03
- added J3: ESC_L, Connector_PinSocket_2.54mm:PinSocket_1x03_P2.54mm_Vertical, symbol Connector_Generic:Conn_01x03
- added J4: Conn_02x08_Odd_Even, Connector_PinSocket_2.54mm:PinSocket_2x08_P2.54mm_Vertical, symbol Connector_Generic:Conn_02x08_Odd_Even
- added J7: ESC_R, Connector_PinSocket_2.54mm:PinSocket_1x03_P2.54mm_Vertical, symbol Connector_Generic:Conn_01x03
- added R22, R23, R25, R26, R27: 10k, Resistor_SMD:R_0805_2012Metric_Pad1.20x1.40mm_HandSolder, symbol Device:R_US
- added R24: 20k, Resistor_SMD:R_0805_2012Metric_Pad1.20x1.40mm_HandSolder, symbol Device:R_US
- added SW1: SW_Push, Button_Switch_SMD:SW_SPST_PTS810, symbol Switch:SW_Push
- added U4: ESP32-S3-WROOM-1, dolphin:ESP32-S3-WROOM-1, symbol RF_Module:ESP32-S3-WROOM-1
Connections:
- net +3V3: now also C9.2, J4.2 (Pin_2), R22.1, R25.1, R26.1, R27.2, U4.2 (3V3)
- net +5V: now also J1.2 (Pin_2), J3.2 (Pin_2), J4.1 (Pin_1), J7.2 (Pin_2)
- net GND: now also C10.2, C9.1, J1.1 (Pin_1), J3.1 (Pin_1), J4.3 (Pin_3), J4.4 (Pin_4), J7.1 (Pin_1), R24.2, SW1.1, U4.1 (GND), U4.40 (GND), U4.41 (GND)
- net USB_D+: now also U4.14 (IO20)
- net USB_D-: now also U4.13 (IO19)
- new net ENC_L_3V3: U4.24 (IO47)
- new net ENC_R_3V3: U4.17 (IO9)
- new net ESC_L_3V3: J3.3 (Pin_3), U4.25 (IO48)
- new net ESC_R_3V3: J7.3 (Pin_3), U4.12 (IO8)
- new net I2C_SCL: J4.13 (Pin_13), R25.2, U4.10 (IO17)
- new net I2C_SDA: J4.15 (Pin_15), R26.2, U4.11 (IO18)
- new net IO00_3V3: J4.6 (Pin_6), R27.1, U4.27 (IO0)
- new net IO10_3V3: J4.16 (Pin_16), U4.18 (IO10)
- new net IO21_3V3: J4.14 (Pin_14), U4.23 (IO21)
- new net IO35_3V3: J4.8 (Pin_8), U4.28 (IO35)
- new net IO36_3V3: J4.12 (Pin_12), U4.29 (IO36)
- new net IO37_3V3: J4.10 (Pin_10), U4.30 (IO37)
- new net LRGB_3V3: U4.4 (IO4)
- new net MS_IR_3V3: R23.2, R24.1, U4.39 (IO1)
- new net MS_IR_5V: J1.3 (Pin_3), R23.1
- new net MUX_COMM_3V3: U4.9 (IO16)
- new net MUX_SEL0: U4.7 (IO7)
- new net MUX_SEL1: U4.8 (IO15)
- new net MUX_SEL2: U4.5 (IO5)
- new net MUX_SEL3: U4.6 (IO6)
- new net NRST: C10.1, R22.2, SW1.2, U4.3 (EN)
- new net RC_CH1_3V3: U4.38 (IO2)
- new net RC_CH2_3V3: U4.35 (IO42)
- new net RC_CH3_3V3: U4.34 (IO41)
- new net RC_CH4_3V3: U4.33 (IO40)
- new net RC_CH5_3V3: U4.32 (IO39)
- new net RC_CH6_3V3: U4.31 (IO38)
- new net SPI_CSn: J4.5 (Pin_5), U4.22 (IO14)
- new net SPI_MISO: J4.7 (Pin_7), U4.21 (IO13)
- new net SPI_MOSI: J4.11 (Pin_11), U4.19 (IO11)
- new net SPI_SCLK: J4.9 (Pin_9), U4.20 (IO12)
- no-connect marks 0 -> 5
Other:
- note added: "booting circuit"
- note added: "decoupling"
- note added: "resetting circuit"

Commit message: chore: rename schematic sheets
Other:
- title: dolphin -> dolphin/mainboard/processor
Changed lines of the file:
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@@
 	(paper "A4")
 	(title_block
-		(title "dolphin")
+		(title "dolphin/mainboard/processor")
 		(date "2026-08-03")
 		(rev "v2")
