File: hardware/projects/mainboard/radio.kicad_sch (KiCad schematic)
At the start: 13 parts

Commit message: chore: rename schematic sheets
Other:
- title: dolphin -> dolphin/mainboard/radio
Changed lines of the file:
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@@
 	(paper "A4")
 	(title_block
-		(title "dolphin")
+		(title "dolphin/mainboard/radio")
 		(date "2026-08-03")
 		(rev "v2")
