File: hardware/projects/mainboard/sensors.kicad_sch (KiCad schematic)
At the start: 29 parts, among them J8 ENC_R, J9 ENC_L, U3 CD74HC4067M

Commit message: chore: rename schematic sheets
Other:
- title: dolphin -> dolphin/mainboard/sensors
Changed lines of the file:
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@@
 	(paper "A4")
 	(title_block
-		(title "dolphin")
+		(title "dolphin/mainboard/sensors")
 		(date "2026-08-03")
 		(rev "v2")
